File: KiCad/KikaiBoard/KikaiBoard.sch (KiCad schematic (older format))
At the start: 1 part

Commit message: Add LFE5U85
Parts:
- added J?: USB4105-GF-A, USB4105-GF-A_GCT, symbol USB4105-GF-A:USB4105-GF-A
- added U? (x3): LFE5U-85F-8MG285I, CSFBGA285_LAT, symbol LFE5U-85F:LFE5U-85F-8MG285I
Other:
- moved on the sheet: U?
Changed lines of the file:
@@
 L BQ25792:PQ25792RQMR U?
 U 1 1 6129E88D
-P 4750 2650
-F 0 "U?" H 5650 3038 60  0000 C CNN
-F 1 "PQ25792RQMR" H 5650 2932 60  0000 C CNN
-F 2 "RQM0029A-MFG" H 4750 2590 60  0001 C CNN
-F 3 "" H 4750 2650 60  0000 C CNN
-	1    4750 2650
+P 800 2600
+F 0 "U?" H 1700 2988 60  0000 C CNN
+F 1 "PQ25792RQMR" H 1700 2882 60  0000 C CNN
+F 2 "RQM0029A-MFG" H 800 2540 60  0001 C CNN
+F 3 "" H 800 2600 60  0000 C CNN
+	1    800  2600
 	1    0    0    -1
 $EndComp
+$Comp
+L USB4105-GF-A:USB4105-GF-A J?
+U 1 1 612A4D45
+P 800 1250
+F 0 "J?" H 1600 1637 60  0000 C CNN
+F 1 "USB4105-GF-A" H 1600 1531 60  0000 C CNN
+F 2 "USB4105-GF-A_GCT" H 1600 1490 60  0001 C CNN
+F 3 "" H 800 1250 60  0000 C CNN
+	1    800  1250
+	1    0    0    -1
+$EndComp
+$Comp
+L LFE5U-85F:LFE5U-85F-8MG285I U?
+U 1 1 612EB01D
+P 2900 1050
+F 0 "U?" H 3900 1437 60  0000 C CNN
+F 1 "LFE5U-85F-8MG285I" H 3900 1331 60  0000 C CNN
+F 2 "CSFBGA285_LAT" H 3900 1290 60  0001 C CNN
+F 3 "" H 2900 1050 60  0000 C CNN
+	1    2900 1050
+	1    0    0    -1
+$EndComp
+$Comp
+L LFE5U-85F:LFE5U-85F-8MG285I U?
+U 2 1 612EEFF3
+P 5150 1050
+F 0 "U?" H 6150 1437 60  0000 C CNN
+F 1 "LFE5U-85F-8MG285I" H 6150 1331 60  0000 C CNN
+F 2 "CSFBGA285_LAT" H 6150 1290 60  0001 C CNN
+F 3 "" H 5150 1050 60  0000 C CNN
+	2    5150 1050
+	1    0    0    -1
+$EndComp
+$Comp
+L LFE5U-85F:LFE5U-85F-8MG285I U?
+U 3 1 612FD708
+P 7400 1050
+F 0 "U?" H 8400 1437 60  0000 C CNN
+F 1 "LFE5U-85F-8MG285I" H 8400 1331 60  0000 C CNN
+F 2 "CSFBGA285_LAT" H 8400 1290 60  0001 C CNN
+F 3 "" H 7400 1050 60  0000 C CNN
+	3    7400 1050
+	1    0    0    -1
+$EndComp
