File: KiCad/power-2.5V.kicad_sch (KiCad schematic)
At the start: 1 part

Commit message: chore(pcb): start from scratch using TPSM63606RDLR
Parts:
- removed U?: TPS84320RUQR, RUQ_47, symbol Buck converter:TPS84320RUQR
Changed lines of the file:
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@@
 (kicad_sch (version 20211123) (generator eeschema)
   (paper "A4")
-  (junction (at 170.688 68.3768) (diameter 0) (color 0 0 0 0)
-  )
-  (junction (at 170.688 81.0768) (diameter 0) (color 0 0 0 0)
-  )
-  (junction (at 170.688 70.9168) (diameter 0) (color 0 0 0 0)
-  )
-  (junction (at 170.688 73.4568) (diameter 0) (color 0 0 0 0)
-  )
-  (junction (at 170.688 78.5368) (diameter 0) (color 0 0 0 0)
-  )
-  (junction (at 170.688 75.9968) (diameter 0) (color 0 0 0 0)
-  )
-  (junction (at 170.688 65.8368) (diameter 0) (color 0 0 0 0)
-  )
-  (wire (pts (xy 170.688 81.0768) (xy 170.688 83.6168))
-    (stroke (width 0) (type default) (color 0 0 0 0))
-  )
-  (wire (pts (xy 170.688 73.4568) (xy 170.688 75.9968))
-    (stroke (width 0) (type default) (color 0 0 0 0))
-  )
-  (wire (pts (xy 170.688 70.9168) (xy 170.688 73.4568))
-    (stroke (width 0) (type default) (color 0 0 0 0))
-  )
-  (wire (pts (xy 170.688 63.2968) (xy 170.688 65.8368))
-    (stroke (width 0) (type default) (color 0 0 0 0))
-  )
-  (wire (pts (xy 170.688 78.5368) (xy 170.688 81.0768))
-    (stroke (width 0) (type default) (color 0 0 0 0))
-  )
-  (wire (pts (xy 170.688 63.2968) (xy 173.228 63.2968))
-    (stroke (width 0) (type default) (color 0 0 0 0))
-  )
-  (wire (pts (xy 170.688 65.8368) (xy 170.688 68.3768))
-    (stroke (width 0) (type default) (color 0 0 0 0))
-  )
-  (wire (pts (xy 170.688 75.9968) (xy 170.688 78.5368))
-    (stroke (width 0) (type default) (color 0 0 0 0))
-  )
-  (wire (pts (xy 170.688 68.3768) (xy 170.688 70.9168))
-    (stroke (width 0) (type default) (color 0 0 0 0))
-  )
-  (global_label "2V5" (shape input) (at 173.228 63.2968 0) (fields_autoplaced)
-    (effects (font (size 1.27 1.27)) (justify left))
-    (property "Intersheet References" "${INTERSHEET_REFS}" (id 0) (at 179.1487 63.2174 0)
-      (effects (font (size 1.27 1.27)) (justify left) hide)
-    )
-  )
-  (symbol (lib_id "Buck converter:TPS84320RUQR") (at 119.888 55.6768 0) (unit 1)
-    (in_bom yes) (on_board yes) (fields_autoplaced)
-    (property "Reference" "U?" (id 0) (at 145.288 44.2468 0)
-      (effects (font (size 1.524 1.524)))
-    )
-    (property "Value" "TPS84320RUQR" (id 1) (at 145.288 48.0568 0)
-      (effects (font (size 1.524 1.524)))
-    )
-    (property "Footprint" "RUQ_47" (id 2) (at 145.288 49.5808 0)
-      (effects (font (size 1.524 1.524)) hide)
-    )
-    (property "Datasheet" "" (id 3) (at 119.888 55.6768 0)
-      (effects (font (size 1.524 1.524)))
-    )
-    (pin "1")
-    (pin "10")
-    (pin "11")
-    (pin "12")
-    (pin "13")
-    (pin "14")
-    (pin "15")
-    (pin "16")
-    (pin "17")
-    (pin "18")
-    (pin "19")
-    (pin "2")
-    (pin "20")
-    (pin "21")
-    (pin "22")
-    (pin "23")
-    (pin "24")
-    (pin "25")
-    (pin "26")
-    (pin "27")
-    (pin "28")
-    (pin "29")
-    (pin "3")
-    (pin "30")
-    (pin "31")
-    (pin "32")
-    (pin "33")
-    (pin "34")
-    (pin "35")
-    (pin "36")
-    (pin "37")
-    (pin "38")
-    (pin "39")
-    (pin "4")
-    (pin "40")
-    (pin "41")
-    (pin "42")
-    (pin "43")
-    (pin "44")
-    (pin "45")
-    (pin "46")
-    (pin "47")
-    (pin "5")
-    (pin "6")
-    (pin "7")
-    (pin "8")
-    (pin "9")
-  )
 )

Commit message: chore(pcb): split voltage regulators to separate schematics
Parts:
- added U?: TPS84320RUQR, RUQ_47, symbol Buck converter:TPS84320RUQR
Connections:
- new net 2V5: U?.21 (VO), U?.24 (VO), U?.25 (VO), U?.26 (VO), U?.27 (VO), U?.28 (VO), U?.29 (VO), U?.47 (VO)
Changed lines of the file:
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@@
 (kicad_sch (version 20211123) (generator eeschema)
   (paper "A4")
+  (junction (at 170.688 68.3768) (diameter 0) (color 0 0 0 0)
+  )
+  (junction (at 170.688 81.0768) (diameter 0) (color 0 0 0 0)
+  )
+  (junction (at 170.688 70.9168) (diameter 0) (color 0 0 0 0)
+  )
+  (junction (at 170.688 73.4568) (diameter 0) (color 0 0 0 0)
+  )
+  (junction (at 170.688 78.5368) (diameter 0) (color 0 0 0 0)
+  )
+  (junction (at 170.688 75.9968) (diameter 0) (color 0 0 0 0)
+  )
+  (junction (at 170.688 65.8368) (diameter 0) (color 0 0 0 0)
+  )
+  (wire (pts (xy 170.688 81.0768) (xy 170.688 83.6168))
+    (stroke (width 0) (type default) (color 0 0 0 0))
+  )
+  (wire (pts (xy 170.688 73.4568) (xy 170.688 75.9968))
+    (stroke (width 0) (type default) (color 0 0 0 0))
+  )
+  (wire (pts (xy 170.688 70.9168) (xy 170.688 73.4568))
+    (stroke (width 0) (type default) (color 0 0 0 0))
+  )
+  (wire (pts (xy 170.688 63.2968) (xy 170.688 65.8368))
+    (stroke (width 0) (type default) (color 0 0 0 0))
+  )
+  (wire (pts (xy 170.688 78.5368) (xy 170.688 81.0768))
+    (stroke (width 0) (type default) (color 0 0 0 0))
+  )
+  (wire (pts (xy 170.688 63.2968) (xy 173.228 63.2968))
+    (stroke (width 0) (type default) (color 0 0 0 0))
+  )
+  (wire (pts (xy 170.688 65.8368) (xy 170.688 68.3768))
+    (stroke (width 0) (type default) (color 0 0 0 0))
+  )
+  (wire (pts (xy 170.688 75.9968) (xy 170.688 78.5368))
+    (stroke (width 0) (type default) (color 0 0 0 0))
+  )
+  (wire (pts (xy 170.688 68.3768) (xy 170.688 70.9168))
+    (stroke (width 0) (type default) (color 0 0 0 0))
+  )
+  (global_label "2V5" (shape input) (at 173.228 63.2968 0) (fields_autoplaced)
+    (effects (font (size 1.27 1.27)) (justify left))
+    (property "Intersheet References" "${INTERSHEET_REFS}" (id 0) (at 179.1487 63.2174 0)
+      (effects (font (size 1.27 1.27)) (justify left) hide)
+    )
+  )
+  (symbol (lib_id "Buck converter:TPS84320RUQR") (at 119.888 55.6768 0) (unit 1)
+    (in_bom yes) (on_board yes) (fields_autoplaced)
+    (property "Reference" "U?" (id 0) (at 145.288 44.2468 0)
+      (effects (font (size 1.524 1.524)))
+    )
+    (property "Value" "TPS84320RUQR" (id 1) (at 145.288 48.0568 0)
+      (effects (font (size 1.524 1.524)))
+    )
+    (property "Footprint" "RUQ_47" (id 2) (at 145.288 49.5808 0)
+      (effects (font (size 1.524 1.524)) hide)
+    )
+    (property "Datasheet" "" (id 3) (at 119.888 55.6768 0)
+      (effects (font (size 1.524 1.524)))
+    )
+    (pin "1")
+    (pin "10")
+    (pin "11")
+    (pin "12")
+    (pin "13")
+    (pin "14")
+    (pin "15")
+    (pin "16")
+    (pin "17")
+    (pin "18")
+    (pin "19")
+    (pin "2")
+    (pin "20")
+    (pin "21")
+    (pin "22")
+    (pin "23")
+    (pin "24")
+    (pin "25")
+    (pin "26")
+    (pin "27")
+    (pin "28")
+    (pin "29")
+    (pin "3")
+    (pin "30")
+    (pin "31")
+    (pin "32")
+    (pin "33")
+    (pin "34")
+    (pin "35")
+    (pin "36")
+    (pin "37")
+    (pin "38")
+    (pin "39")
+    (pin "4")
+    (pin "40")
+    (pin "41")
+    (pin "42")
+    (pin "43")
+    (pin "44")
+    (pin "45")
+    (pin "46")
+    (pin "47")
+    (pin "5")
+    (pin "6")
+    (pin "7")
+    (pin "8")
+    (pin "9")
+  )
 )
