File: KiCad/flash.kicad_sch (KiCad schematic)
At the start: 1 part

Commit message: chore(pcb): start from scratch using TPSM63606RDLR
Parts:
- removed IC?: W25Q128JVPIQ, SON127P800X600X80-9N-D, symbol SPI Flash:W25Q128JVPIQ
Changed lines of the file:
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@@
 (kicad_sch (version 20211123) (generator eeschema)
   (paper "A4")
-  (symbol (lib_id "SPI Flash:W25Q128JVPIQ") (at 49.53 44.45 0) (unit 1)
-    (in_bom yes) (on_board yes) (fields_autoplaced)
-    (property "Reference" "IC?" (id 0) (at 67.31 36.83 0))
-    (property "Value" "W25Q128JVPIQ" (id 1) (at 67.31 39.37 0))
-    (property "Footprint" "SON127P800X600X80-9N-D" (id 2) (at 81.28 41.91 0)
-      (effects (font (size 1.27 1.27)) (justify left) hide)
-    )
-    (property "Datasheet" "https://www.arrow.com/en/products/w25q128jvpiq/winbond-electronics" (id 3) (at 81.28 44.45 0)
-      (effects (font (size 1.27 1.27)) (justify left) hide)
-    )
-    (property "Description" "IC FLASH 128M SPI 133MHZ 8WSON" (id 4) (at 81.28 46.99 0)
-      (effects (font (size 1.27 1.27)) (justify left) hide)
-    )
-    (property "Height" "0.8" (id 5) (at 81.28 49.53 0)
-      (effects (font (size 1.27 1.27)) (justify left) hide)
-    )
-    (property "Mouser Part Number" "454-W25Q128JVPIQ" (id 6) (at 81.28 52.07 0)
-      (effects (font (size 1.27 1.27)) (justify left) hide)
-    )
-    (property "Mouser Price/Stock" "https://www.mouser.co.uk/ProductDetail/Winbond/W25Q128JVPIQ?qs=qSfuJ%252Bfl%2Fd676hAD%252B1JSfw%3D%3D" (id 7) (at 81.28 54.61 0)
-      (effects (font (size 1.27 1.27)) (justify left) hide)
-    )
-    (property "Manufacturer_Name" "Winbond" (id 8) (at 81.28 57.15 0)
-      (effects (font (size 1.27 1.27)) (justify left) hide)
-    )
-    (property "Manufacturer_Part_Number" "W25Q128JVPIQ" (id 9) (at 81.28 59.69 0)
-      (effects (font (size 1.27 1.27)) (justify left) hide)
-    )
-    (pin "1")
-    (pin "2")
-    (pin "3")
-    (pin "4")
-    (pin "5")
-    (pin "6")
-    (pin "7")
-    (pin "8")
-    (pin "9")
-  )
 )
