File: KiCad/fpga.kicad_sch (KiCad schematic)
At the start: 9 parts

Commit message: chore(pcb): start from scratch using TPSM63606RDLR
Parts:
- removed U? (x7): ECP5U_85_CSFBGA285, symbol ECP5:ECP5U_85_CSFBGA285
- removed U? (x2): ECP5U_85_CSFBGA285, ECP5:BGA285C50P18X18_1000X1000X130, symbol ECP5:ECP5U_85_CSFBGA285
