File: KiCad/logic-level-conversion.kicad_sch (KiCad schematic)
At the start: 1 part

Commit message: chore(pcb): start from scratch using TPSM63606RDLR
Parts:
- removed IC?: LSF0204DYZPR, BGA12C50P3X4_144X194X50, symbol Voltage Level Translator:LSF0204DYZPR
Changed lines of the file:
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@@
 (kicad_sch (version 20211123) (generator eeschema)
   (paper "A4")
-  (symbol (lib_id "Voltage Level Translator:LSF0204DYZPR") (at 44.45 39.37 0) (unit 1)
-    (in_bom yes) (on_board yes) (fields_autoplaced)
-    (property "Reference" "IC?" (id 0) (at 59.69 31.6992 0))
-    (property "Value" "LSF0204DYZPR" (id 1) (at 59.69 34.2392 0))
-    (property "Footprint" "BGA12C50P3X4_144X194X50" (id 2) (at 71.12 36.83 0)
-      (effects (font (size 1.27 1.27)) (justify left) hide)
-    )
-    (property "Datasheet" "http://www.ti.com/lit/gpn/lsf0204d" (id 3) (at 71.12 39.37 0)
-      (effects (font (size 1.27 1.27)) (justify left) hide)
-    )
-    (property "Description" "4-Bit Bidirectional Multi-Voltage Level Translator for Open-Drain & Push-Pull" (id 4) (at 71.12 41.91 0)
-      (effects (font (size 1.27 1.27)) (justify left) hide)
-    )
-    (property "Height" "0.5" (id 5) (at 71.12 44.45 0)
-      (effects (font (size 1.27 1.27)) (justify left) hide)
-    )
-    (property "Mouser Part Number" "595-LSF0204DYZPR" (id 6) (at 71.12 46.99 0)
-      (effects (font (size 1.27 1.27)) (justify left) hide)
-    )
-    (property "Mouser Price/Stock" "https://www.mouser.co.uk/ProductDetail/Texas-Instruments/LSF0204DYZPR?qs=UfUFg%2FkmHHHXMV6u4PWobw%3D%3D" (id 7) (at 71.12 49.53 0)
-      (effects (font (size 1.27 1.27)) (justify left) hide)
-    )
-    (property "Manufacturer_Name" "Texas Instruments" (id 8) (at 71.12 52.07 0)
-      (effects (font (size 1.27 1.27)) (justify left) hide)
-    )
-    (property "Manufacturer_Part_Number" "LSF0204DYZPR" (id 9) (at 71.12 54.61 0)
-      (effects (font (size 1.27 1.27)) (justify left) hide)
-    )
-    (pin "A1")
-    (pin "A2")
-    (pin "A3")
-    (pin "B1")
-    (pin "B2")
-    (pin "B3")
-    (pin "C1")
-    (pin "C2")
-    (pin "C3")
-    (pin "D1")
-    (pin "D2")
-    (pin "D3")
-  )
 )
