File: KiCad/power-1.1V.kicad_sch (KiCad schematic)
At the start: 4 parts

Commit message: chore(pcb): split voltage regulators to separate schematics
Parts:
- removed U? (x2): TPS84320RUQR, RUQ_47, symbol Buck converter:TPS84320RUQR
Other:
- moved on the sheet: R?, U?

Commit message: chore(pcb): start from scratch using TPSM63606RDLR
Parts:
- removed R?: 866, symbol Device:R
- removed U?: TPSM84A21MOJR, Texas_Instruments-MOJ0020A-0-0-*, symbol Buck (build-in caps):TPSM84A21MOJR
Changed lines of the file:
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@@
 (kicad_sch (version 20211123) (generator eeschema)
   (paper "A4")
-  (wire (pts (xy 133.096 88.138) (xy 135.636 88.138))
-    (stroke (width 0) (type default) (color 0 0 0 0))
-  )
-  (wire (pts (xy 122.936 88.138) (xy 125.476 88.138))
-    (stroke (width 0) (type default) (color 0 0 0 0))
-  )
-  (wire (pts (xy 171.196 77.978) (xy 173.736 77.978))
-    (stroke (width 0) (type default) (color 0 0 0 0))
-  )
-  (global_label "1V1" (shape input) (at 173.736 77.978 0) (fields_autoplaced)
-    (effects (font (size 1.27 1.27)) (justify left))
-    (property "Intersheet References" "${INTERSHEET_REFS}" (id 0) (at 179.6567 77.8986 0)
-      (effects (font (size 1.27 1.27)) (justify left) hide)
-    )
-  )
-  (symbol (lib_id "power:GND") (at 122.936 88.138 270) (unit 1)
-    (in_bom yes) (on_board yes) (fields_autoplaced)
-    (property "Reference" "#PWR?" (id 0) (at 116.586 88.138 0)
-      (effects (font (size 1.27 1.27)) hide)
-    )
-    (property "Value" "GND" (id 1) (at 119.126 88.1379 90)
-      (effects (font (size 1.27 1.27)) (justify right))
-    )
-    (property "Footprint" "" (id 2) (at 122.936 88.138 0)
-      (effects (font (size 1.27 1.27)) hide)
-    )
-    (property "Datasheet" "" (id 3) (at 122.936 88.138 0)
-      (effects (font (size 1.27 1.27)) hide)
-    )
-    (pin "1")
-  )
-  (symbol (lib_id "Buck (build-in caps):TPSM84A21MOJR") (at 133.096 77.978 0) (unit 1)
-    (in_bom yes) (on_board yes) (fields_autoplaced)
-    (property "Reference" "U?" (id 0) (at 153.416 70.358 0))
-    (property "Value" "TPSM84A21MOJR" (id 1) (at 153.416 72.898 0))
-    (property "Footprint" "Texas_Instruments-MOJ0020A-0-0-*" (id 2) (at 133.096 67.818 0)
-      (effects (font (size 1.27 1.27)) (justify left) hide)
-    )
-    (property "Datasheet" "https://www.ti.com/lit/ds/symlink/tpsm84a21.pdf?ts=1616475331887&ref_url=https%253A%252F%252Fwww.ti.com%252Fproduct%252FTPSM84A21%253FkeyMatch%253DTPSM84A21MOJR%2526tisearch%253Dsearch-everything%2526usecase%253DOPN" (id 3) (at 133.096 65.278 0)
-      (effects (font (size 1.27 1.27)) (justify left) hide)
-    )
-    (property "ambient temperature range high" "+85°C" (id 4) (at 133.096 62.738 0)
-      (effects (font (size 1.27 1.27)) (justify left) hide)
-    )
-    (property "ambient temperature range low" "-40°C" (id 5) (at 133.096 60.198 0)
-      (effects (font (size 1.27 1.27)) (justify left) hide)
-    )
-    (property "automotive" "No" (id 6) (at 133.096 57.658 0)
-      (effects (font (size 1.27 1.27)) (justify left) hide)
-    )
-    (property "category" "IC" (id 7) (at 133.096 55.118 0)
-      (effects (font (size 1.27 1.27)) (justify left) hide)
-    )
-    (property "device class L1" "Integrated Circuits (ICs)" (id 8) (at 133.096 52.578 0)
-      (effects (font (size 1.27 1.27)) (justify left) hide)
-    )
-    (property "device class L2" "Power Management ICs" (id 9) (at 133.096 50.038 0)
-      (effects (font (size 1.27 1.27)) (justify left) hide)
-    )
-    (property "device class L3" "Voltage Regulators - Switching" (id 10) (at 133.096 47.498 0)
-      (effects (font (size 1.27 1.27)) (justify left) hide)
-    )
-    (property "digikey description" "DC DC CONVERTER 0.55-1.35V" (id 11) (at 133.096 44.958 0)
-      (effects (font (size 1.27 1.27)) (justify left) hide)
-    )
-    (property "digikey part number" "296-48785-1-ND" (id 12) (at 133.096 42.418 0)
-      (effects (font (size 1.27 1.27)) (justify left) hide)
-    )
-    (property "height" "2.3mm" (id 13) (at 133.096 39.878 0)
-      (effects (font (size 1.27 1.27)) (justify left) hide)
-    )
-    (property "ipc land pattern name" "CAPAD1016W80L630D240" (id 14) (at 133.096 37.338 0)
-      (effects (font (size 1.27 1.27)) (justify left) hide)
-    )
-    (property "lead free" "Yes" (id 15) (at 133.096 34.798 0)
-      (effects (font (size 1.27 1.27)) (justify left) hide)
-    )
-    (property "library id" "cebd5fe4464742bf" (id 16) (at 133.096 32.258 0)
-      (effects (font (size 1.27 1.27)) (justify left) hide)
-    )
-    (property "manufacturer" "Texas Instruments" (id 17) (at 133.096 29.718 0)
-      (effects (font (size 1.27 1.27)) (justify left) hide)
-    )
-    (property "max duty cycle" "80%" (id 18) (at 133.096 27.178 0)
-      (effects (font (size 1.27 1.27)) (justify left) hide)
-    )
-    (property "max junction temp" "+125°C" (id 19) (at 133.096 24.638 0)
-      (effects (font (size 1.27 1.27)) (justify left) hide)
-    )
-    (property "max supply voltage" "14V" (id 20) (at 133.096 22.098 0)
-      (effects (font (size 1.27 1.27)) (justify left) hide)
-    )
-    (property "min supply voltage" "8V" (id 21) (at 133.096 19.558 0)
-      (effects (font (size 1.27 1.27)) (justify left) hide)
-    )
-    (property "mouser description" "8V to 14V, 0.508V to 1.35V Output, 10A Power Module with Integrated Input and Output Capacitors 20-QFM -40 to 85" (id 22) (at 133.096 17.018 0)
-      (effects (font (size 1.27 1.27)) (justify left) hide)
-    )
-    (property "mouser part number" "595-TPSM84A21MOJR" (id 23) (at 133.096 14.478 0)
-      (effects (font (size 1.27 1.27)) (justify left) hide)
-    )
-    (property "nominal supply current" "8mA" (id 24) (at 133.096 11.938 0)
-      (effects (font (size 1.27 1.27)) (justify left) hide)
-    )
-    (property "number of outputs" "1" (id 25) (at 133.096 9.398 0)
-      (effects (font (size 1.27 1.27)) (justify left) hide)
-    )
-    (property "output current" "10A" (id 26) (at 133.096 6.858 0)
-      (effects (font (size 1.27 1.27)) (justify left) hide)
-    )
-    (property "output type" "AdjustableProgrammable" (id 27) (at 133.096 4.318 0)
-      (effects (font (size 1.27 1.27)) (justify left) hide)
-    )
-    (property "output voltage" "0.55-1.35V" (id 28) (at 133.096 1.778 0)
-      (effects (font (size 1.27 1.27)) (justify left) hide)
-    )
-    (property "package" "QFM20" (id 29) (at 133.096 -0.762 0)
-      (effects (font (size 1.27 1.27)) (justify left) hide)
-    )
-    (property "rohs" "Yes" (id 30) (at 133.096 -3.302 0)
-      (effects (font (size 1.27 1.27)) (justify left) hide)
-    )
-    (property "switching frequency" "4MHz" (id 31) (at 133.096 -5.842 0)
-      (effects (font (size 1.27 1.27)) (justify left) hide)
-    )
-    (property "temperature range high" "+85°C" (id 32) (at 133.096 -8.382 0)
-      (effects (font (size 1.27 1.27)) (justify left) hide)
-    )
-    (property "temperature range low" "-40°C" (id 33) (at 133.096 -10.922 0)
-      (effects (font (size 1.27 1.27)) (justify left) hide)
-    )
-    (pin "1")
-    (pin "10")
-    (pin "11")
-    (pin "12")
-    (pin "13")
-    (pin "14")
-    (pin "15")
-    (pin "16")
-    (pin "17")
-    (pin "18")
-    (pin "19")
-    (pin "2")
-    (pin "20")
-    (pin "3")
-    (pin "4")
-    (pin "5")
-    (pin "6")
-    (pin "7")
-    (pin "8")
-    (pin "9")
-  )
-  (symbol (lib_id "Device:R") (at 129.286 88.138 90) (unit 1)
-    (in_bom yes) (on_board yes) (fields_autoplaced)
-    (property "Reference" "R?" (id 0) (at 129.286 81.788 90))
-    (property "Value" "866" (id 1) (at 129.286 84.328 90))
-    (property "Footprint" "" (id 2) (at 129.286 89.916 90)
-      (effects (font (size 1.27 1.27)) hide)
-    )
-    (property "Datasheet" "~" (id 3) (at 129.286 88.138 0)
-      (effects (font (size 1.27 1.27)) hide)
-    )
-    (pin "1")
-    (pin "2")
-  )
 )
