File: KiCad/power-3.3V.kicad_sch (KiCad schematic)
At the start: 8 parts

Commit message: feat(pcb): add passives to 3.3V power schematic
Parts:
- C?: footprint (none) -> Capacitor_SMD:C_1210_3225Metric
Connections:
- no-connect marks 0 -> 5
Changed lines of the file:
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@@
   (junction (at 170.18 69.85) (diameter 0) (color 0 0 0 0)
   )
+  (no_connect (at 119.38 69.85))
+  (no_connect (at 119.38 74.93))
+  (no_connect (at 119.38 64.77))
+  (no_connect (at 119.38 62.23))
+  (no_connect (at 119.38 128.27))
   (wire (pts (xy 170.18 85.09) (xy 170.18 87.63))
     (stroke (width 0) (type default) (color 0 0 0 0))
@@
       (effects (font (size 1.27 1.27)) (justify right))
     )
-    (property "Footprint" "" (id 2) (at 111.76 91.44 0)
-      (effects (font (size 1.27 1.27)) hide)
-    )
-    (property "Datasheet" "~" (id 3) (at 111.76 91.44 0)
-      (effects (font (size 1.27 1.27)) hide)
-    )
+    (property "Footprint" "Capacitor_SMD:C_1210_3225Metric" (id 2) (at 111.76 91.44 0)
+      (effects (font (size 1.27 1.27)) hide)
+    )
+    (property "Datasheet" "https://www.mouser.co.uk/datasheet/2/281/1/GRM32ER61E226KE15_01A-1988202.pdf" (id 3) (at 111.76 91.44 0)
+      (effects (font (size 1.27 1.27)) hide)
+    )

Commit message: chore(pcb): split voltage regulators to separate schematics
Connections:
- net GND: now also U?.7 (STSEL)
- net at U?.10 (PH): now also U?.11 (PH), U?.12 (PH), U?.13 (PH), U?.14 (PH), U?.17 (PH), U?.46 (PH)
- no-connect marks 5 -> 4
Changed lines of the file:
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@@
   (junction (at 170.18 80.01) (diameter 0) (color 0 0 0 0)
   )
+  (junction (at 170.18 97.79) (diameter 0) (color 0 0 0 0)
+  )
   (junction (at 170.18 74.93) (diameter 0) (color 0 0 0 0)
   )
   (junction (at 170.18 85.09) (diameter 0) (color 0 0 0 0)
   )
+  (junction (at 170.18 105.41) (diameter 0) (color 0 0 0 0)
+  )
   (junction (at 193.04 69.85) (diameter 0) (color 0 0 0 0)
   )
@@
   (junction (at 102.87 87.63) (diameter 0) (color 0 0 0 0)
   )
+  (junction (at 170.18 95.25) (diameter 0) (color 0 0 0 0)
+  )
   (junction (at 111.76 87.63) (diameter 0) (color 0 0 0 0)
   )
@@
   )
   (junction (at 119.38 82.55) (diameter 0) (color 0 0 0 0)
+  )
+  (junction (at 170.18 100.33) (diameter 0) (color 0 0 0 0)
+  )
+  (junction (at 170.18 102.87) (diameter 0) (color 0 0 0 0)
   )
   (junction (at 189.23 69.85) (diameter 0) (color 0 0 0 0)
@@
   (no_connect (at 119.38 74.93))
   (no_connect (at 119.38 64.77))
-  (no_connect (at 119.38 62.23))
   (no_connect (at 119.38 128.27))
   (wire (pts (xy 170.18 85.09) (xy 170.18 87.63))
@@
     (stroke (width 0) (type default) (color 0 0 0 0))
   )
+  (wire (pts (xy 170.18 100.33) (xy 170.18 102.87))
+    (stroke (width 0) (type default) (color 0 0 0 0))
+  )
   (wire (pts (xy 118.11 59.69) (xy 119.38 59.69))
     (stroke (width 0) (type default) (color 0 0 0 0))
@@
     (stroke (width 0) (type default) (color 0 0 0 0))
   )
+  (wire (pts (xy 170.18 97.79) (xy 170.18 100.33))
+    (stroke (width 0) (type default) (color 0 0 0 0))
+  )
   (wire (pts (xy 181.61 71.12) (xy 181.61 69.85))
     (stroke (width 0) (type default) (color 0 0 0 0))
@@
     (stroke (width 0) (type default) (color 0 0 0 0))
   )
+  (wire (pts (xy 170.18 92.71) (xy 170.18 95.25))
+    (stroke (width 0) (type default) (color 0 0 0 0))
+  )
   (wire (pts (xy 189.23 69.85) (xy 193.04 69.85))
     (stroke (width 0) (type default) (color 0 0 0 0))
@@
     (stroke (width 0) (type default) (color 0 0 0 0))
   )
+  (wire (pts (xy 118.618 62.23) (xy 119.38 62.23))
+    (stroke (width 0) (type default) (color 0 0 0 0))
+  )
   (wire (pts (xy 170.18 77.47) (xy 170.18 80.01))
     (stroke (width 0) (type default) (color 0 0 0 0))
   )
+  (wire (pts (xy 170.18 95.25) (xy 170.18 97.79))
+    (stroke (width 0) (type default) (color 0 0 0 0))
+  )
   (wire (pts (xy 99.06 67.31) (xy 99.06 45.72))
     (stroke (width 0) (type default) (color 0 0 0 0))
@@
     (stroke (width 0) (type default) (color 0 0 0 0))
   )
+  (wire (pts (xy 170.18 105.41) (xy 170.18 107.95))
+    (stroke (width 0) (type default) (color 0 0 0 0))
+  )
   (wire (pts (xy 111.76 93.98) (xy 111.76 96.52))
     (stroke (width 0) (type default) (color 0 0 0 0))
@@
   )
   (wire (pts (xy 170.18 118.11) (xy 170.18 120.65))
+    (stroke (width 0) (type default) (color 0 0 0 0))
+  )
+  (wire (pts (xy 170.18 102.87) (xy 170.18 105.41))
     (stroke (width 0) (type default) (color 0 0 0 0))
   )
@@
       (effects (font (size 1.27 1.27)) hide)
     )
+    (pin "1")
+  )
+  (symbol (lib_id "power:GND") (at 118.618 62.23 270) (unit 1)
+    (in_bom yes) (on_board yes) (fields_autoplaced)
+    (property "Reference" "#PWR?" (id 0) (at 112.268 62.23 0)
+      (effects (font (size 1.27 1.27)) hide)
+    )
+    (property "Value" "GND" (id 1) (at 114.808 62.2299 90)
+      (effects (font (size 1.27 1.27)) (justify right))
+    )
+    (property "Footprint" "" (id 2) (at 118.618 62.23 0)
+      (effects (font (size 1.27 1.27)) hide)
+    )
+    (property "Datasheet" "" (id 3) (at 118.618 62.23 0)
+      (effects (font (size 1.27 1.27)) hide)
+    )

Commit message: chore(pcb): start from scratch using TPSM63606RDLR
Parts:
- removed C?: 68, symbol Device:C_Polarized_Small_US
- removed C? (x2): 47, symbol Device:C_Small
- removed C?: 22, Capacitor_SMD:C_1210_3225Metric, symbol Device:C_Small
- removed C?: 220, symbol Device:C_Polarized_Small_US
- removed R?: 453, symbol Device:R
- removed R?: 158k, symbol Device:R
- removed U?: TPS84320RUQR, RUQ_47, symbol Buck converter:TPS84320RUQR
Connections:
- no-connect marks 4 -> 0
