File: KiCad/power-5V.kicad_sch (KiCad schematic)
At the start: 3 parts, among them U1 TPSM63606RDLR

Commit message: feat(pcb): add LDO capacitor
Parts:
- added C3: (no value), symbol C1005X6S1C105K050BC:C1005X6S1C105K050BC
Connections:
- net GNDREF: now also C3.1
- net VCC5: now also U1.5 (VLDOIN), C3.2
Changed lines of the file:
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@@
   (junction (at 104.14 129.54) (diameter 0) (color 0 0 0 0)
   )
+  (junction (at 119.38 129.54) (diameter 0) (color 0 0 0 0)
+  )
   (junction (at 177.8 116.84) (diameter 0) (color 0 0 0 0)
   )
@@
   (junction (at 180.34 83.82) (diameter 0) (color 0 0 0 0)
   )
+  (junction (at 127 83.82) (diameter 0) (color 0 0 0 0)
+  )
   (junction (at 104.14 101.6) (diameter 0) (color 0 0 0 0)
   )
+  (junction (at 182.88 83.82) (diameter 0) (color 0 0 0 0)
+  )
   (junction (at 104.14 83.82) (diameter 0) (color 0 0 0 0)
+  )
+  (junction (at 129.54 101.6) (diameter 0) (color 0 0 0 0)
   )
   (junction (at 177.8 121.92) (diameter 0) (color 0 0 0 0)
@@
     (stroke (width 0) (type default) (color 0 0 0 0))
   )
+  (wire (pts (xy 182.88 83.82) (xy 208.28 83.82))
+    (stroke (width 0) (type default) (color 0 0 0 0))
+  )
   (wire (pts (xy 177.8 114.3) (xy 177.8 116.84))
     (stroke (width 0) (type default) (color 0 0 0 0))
   )
+  (wire (pts (xy 119.38 101.6) (xy 119.38 114.3))
+    (stroke (width 0) (type default) (color 0 0 0 0))
+  )
   (wire (pts (xy 177.8 83.82) (xy 180.34 83.82))
     (stroke (width 0) (type default) (color 0 0 0 0))
   )
-  (wire (pts (xy 134.62 91.44) (xy 132.08 91.44))
+  (wire (pts (xy 134.62 91.44) (xy 127 91.44))
     (stroke (width 0) (type default) (color 0 0 0 0))
   )
@@
     (stroke (width 0) (type default) (color 0 0 0 0))
   )
+  (wire (pts (xy 129.54 67.31) (xy 182.88 67.31))
+    (stroke (width 0) (type default) (color 0 0 0 0))
+  )
   (wire (pts (xy 132.08 83.82) (xy 134.62 83.82))
     (stroke (width 0) (type default) (color 0 0 0 0))
@@
     (stroke (width 0) (type default) (color 0 0 0 0))
   )
+  (wire (pts (xy 182.88 67.31) (xy 182.88 83.82))
+    (stroke (width 0) (type default) (color 0 0 0 0))
+  )
   (wire (pts (xy 177.8 109.22) (xy 177.8 111.76))
     (stroke (width 0) (type default) (color 0 0 0 0))
   )
+  (wire (pts (xy 116.84 83.82) (xy 127 83.82))
+    (stroke (width 0) (type default) (color 0 0 0 0))
+  )
   (wire (pts (xy 180.34 81.28) (xy 180.34 83.82))
     (stroke (width 0) (type default) (color 0 0 0 0))
   )
+  (wire (pts (xy 134.62 101.6) (xy 129.54 101.6))
+    (stroke (width 0) (type default) (color 0 0 0 0))
+  )
   (wire (pts (xy 116.84 83.82) (xy 116.84 86.36))
     (stroke (width 0) (type default) (color 0 0 0 0))
   )
-  (wire (pts (xy 116.84 83.82) (xy 132.08 83.82))
-    (stroke (width 0) (type default) (color 0 0 0 0))
-  )
   (wire (pts (xy 177.8 119.38) (xy 177.8 121.92))
     (stroke (width 0) (type default) (color 0 0 0 0))
   )
+  (wire (pts (xy 127 83.82) (xy 132.08 83.82))
+    (stroke (width 0) (type default) (color 0 0 0 0))
+  )
   (wire (pts (xy 104.14 99.06) (xy 104.14 101.6))
     (stroke (width 0) (type default) (color 0 0 0 0))
   )
+  (wire (pts (xy 129.54 101.6) (xy 119.38 101.6))
+    (stroke (width 0) (type default) (color 0 0 0 0))
+  )
   (wire (pts (xy 116.84 101.6) (xy 104.14 101.6))
     (stroke (width 0) (type default) (color 0 0 0 0))
@@
     (stroke (width 0) (type default) (color 0 0 0 0))
   )
+  (wire (pts (xy 129.54 101.6) (xy 129.54 67.31))
+    (stroke (width 0) (type default) (color 0 0 0 0))
+  )
   (wire (pts (xy 104.14 101.6) (xy 104.14 129.54))
     (stroke (width 0) (type default) (color 0 0 0 0))
@@
     (stroke (width 0) (type default) (color 0 0 0 0))
   )
-  (wire (pts (xy 132.08 91.44) (xy 132.08 83.82))
-    (stroke (width 0) (type default) (color 0 0 0 0))
-  )
-  (wire (pts (xy 177.8 129.54) (xy 104.14 129.54))
+  (wire (pts (xy 127 91.44) (xy 127 83.82))
+    (stroke (width 0) (type default) (color 0 0 0 0))
+  )
+  (wire (pts (xy 177.8 129.54) (xy 119.38 129.54))
     (stroke (width 0) (type default) (color 0 0 0 0))
   )
@@
     (stroke (width 0) (type default) (color 0 0 0 0))
   )
+  (wire (pts (xy 119.38 127) (xy 119.38 129.54))
+    (stroke (width 0) (type default) (color 0 0 0 0))
+  )
   (wire (pts (xy 177.8 121.92) (xy 177.8 129.54))
     (stroke (width 0) (type default) (color 0 0 0 0))
@@
     (stroke (width 0) (type default) (color 0 0 0 0))
   )
-  (wire (pts (xy 180.34 83.82) (xy 208.28 83.82))
+  (wire (pts (xy 119.38 129.54) (xy 104.14 129.54))
+    (stroke (width 0) (type default) (color 0 0 0 0))
+  )
+  (wire (pts (xy 180.34 83.82) (xy 182.88 83.82))
     (stroke (width 0) (type default) (color 0 0 0 0))
   )
@@
       (effects (font (size 1.27 1.27)) (justify left) hide)
     )
+    (pin "1")
+    (pin "2")
+  )
+  (symbol (lib_id "C1005X6S1C105K050BC:C1005X6S1C105K050BC") (at 119.38 127 90) (unit 1)
+    (in_bom yes) (on_board yes) (fields_autoplaced)
+    (property "Reference" "C3" (id 0) (at 123.19 119.3799 90)
+      (effects (font (size 1.27 1.27)) (justify right))
+    )
+    (property "Value" "" (id 1) (at 123.19 121.9199 90)
+      (effects (font (size 1.27 1.27)) (justify right))
+    )
+    (property "Footprint" "" (id 2) (at 118.11 118.11 0)
+      (effects (font (size 1.27 1.27)) (justify left) hide)
+    )
+    (property "Datasheet" "https://product.tdk.com/system/files/dam/doc/product/capacitor/ceramic/mlcc/catalog/mlcc_commercial_general_en.pdf" (id 3) (at 120.65 118.11 0)
+      (effects (font (size 1.27 1.27)) (justify left) hide)
+    )
+    (property "Description" "MULTILAYER CERAMIC CHIP CAPACITORS, 1005, Commercial grade, general (Up to 75V)" (id 4) (at 123.19 118.11 0)
+      (effects (font (size 1.27 1.27)) (justify left) hide)
+    )
+    (property "Height" "0.55" (id 5) (at 125.73 118.11 0)
+      (effects (font (size 1.27 1.27)) (justify left) hide)
+    )
+    (property "Mouser Part Number" "810-C1005X6S1C105K" (id 6) (at 128.27 118.11 0)
+      (effects (font (size 1.27 1.27)) (justify left) hide)
+    )
+    (property "Mouser Price/Stock" "https://www.mouser.co.uk/ProductDetail/TDK/C1005X6S1C105K050BC?qs=dfay7wIA1uGWVKHpqb9RWw%3D%3D" (id 7) (at 130.81 118.11 0)
+      (effects (font (size 1.27 1.27)) (justify left) hide)
+    )
+    (property "Manufacturer_Name" "TDK" (id 8) (at 133.35 118.11 0)
+      (effects (font (size 1.27 1.27)) (justify left) hide)
+    )
+    (property "Manufacturer_Part_Number" "C1005X6S1C105K050BC" (id 9) (at 135.89 118.11 0)
+      (effects (font (size 1.27 1.27)) (justify left) hide)
+    )

Commit message: feat(pcb): add resistor for switching frequency
Parts:
- added R1: (no value), symbol Device:R
Connections:
- net GNDREF: now also R1.2
- net at U1.12 (RT): now also R1.1
Changed lines of the file:
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@@
   (junction (at 177.8 116.84) (diameter 0) (color 0 0 0 0)
+  )
+  (junction (at 128.27 129.54) (diameter 0) (color 0 0 0 0)
   )
   (junction (at 177.8 119.38) (diameter 0) (color 0 0 0 0)
@@
     (stroke (width 0) (type default) (color 0 0 0 0))
   )
+  (wire (pts (xy 128.27 127) (xy 128.27 129.54))
+    (stroke (width 0) (type default) (color 0 0 0 0))
+  )
   (wire (pts (xy 182.88 83.82) (xy 208.28 83.82))
     (stroke (width 0) (type default) (color 0 0 0 0))
@@
   )
   (wire (pts (xy 132.08 83.82) (xy 134.62 83.82))
+    (stroke (width 0) (type default) (color 0 0 0 0))
+  )
+  (wire (pts (xy 128.27 129.54) (xy 119.38 129.54))
     (stroke (width 0) (type default) (color 0 0 0 0))
   )
@@
     (stroke (width 0) (type default) (color 0 0 0 0))
   )
-  (wire (pts (xy 177.8 129.54) (xy 119.38 129.54))
+  (wire (pts (xy 128.27 116.84) (xy 128.27 119.38))
+    (stroke (width 0) (type default) (color 0 0 0 0))
+  )
+  (wire (pts (xy 177.8 129.54) (xy 128.27 129.54))
     (stroke (width 0) (type default) (color 0 0 0 0))
   )
@@
     (stroke (width 0) (type default) (color 0 0 0 0))
   )
+  (wire (pts (xy 134.62 116.84) (xy 128.27 116.84))
+    (stroke (width 0) (type default) (color 0 0 0 0))
+  )
   (wire (pts (xy 180.34 83.82) (xy 182.88 83.82))
     (stroke (width 0) (type default) (color 0 0 0 0))
@@
     )
   )
+  (symbol (lib_id "Device:R") (at 128.27 123.19 0) (unit 1)
+    (in_bom yes) (on_board yes) (fields_autoplaced)
+    (property "Reference" "R1" (id 0) (at 130.81 121.9199 0)
+      (effects (font (size 1.27 1.27)) (justify left))
+    )
+    (property "Value" "" (id 1) (at 130.81 124.4599 0)
+      (effects (font (size 1.27 1.27)) (justify left))
+    )
+    (property "Footprint" "" (id 2) (at 126.492 123.19 90)
+      (effects (font (size 1.27 1.27)) hide)
+    )
+    (property "Datasheet" "~" (id 3) (at 128.27 123.19 0)
+      (effects (font (size 1.27 1.27)) hide)
+    )
+    (pin "1")
+    (pin "2")
+  )
   (symbol (lib_id "power:GNDREF") (at 104.14 130.81 0) (unit 1)

Commit message: feat(pcb): add feedback resistors
Parts:
- added R2: (no value), symbol CRCW040240K2FKED:CRCW040240K2FKED
- added R?: (no value), symbol CRCW040210K0FKED:CRCW040210K0FKED
Connections:
- net GNDREF: now also R?.1
- net VCC5: now also R2.2
- net at U1.10 (FB): now also R2.1, R?.2
- net at U1.3 (CBOOT): now also U1.4 (RBOOT)
Changed lines of the file:
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@@
   (junction (at 128.27 129.54) (diameter 0) (color 0 0 0 0)
   )
+  (junction (at 195.58 106.68) (diameter 0) (color 0 0 0 0)
+  )
+  (junction (at 177.8 129.54) (diameter 0) (color 0 0 0 0)
+  )
   (junction (at 177.8 119.38) (diameter 0) (color 0 0 0 0)
   )
@@
   )
   (junction (at 104.14 101.6) (diameter 0) (color 0 0 0 0)
+  )
+  (junction (at 195.58 83.82) (diameter 0) (color 0 0 0 0)
   )
   (junction (at 182.88 83.82) (diameter 0) (color 0 0 0 0)
@@
   (no_connect (at 134.62 111.76))
   (no_connect (at 177.8 104.14))
-  (wire (pts (xy 101.6 83.82) (xy 104.14 83.82))
+  (wire (pts (xy 104.14 81.28) (xy 104.14 83.82))
     (stroke (width 0) (type default) (color 0 0 0 0))
   )
@@
     (stroke (width 0) (type default) (color 0 0 0 0))
   )
-  (wire (pts (xy 182.88 83.82) (xy 208.28 83.82))
+  (wire (pts (xy 182.88 83.82) (xy 195.58 83.82))
+    (stroke (width 0) (type default) (color 0 0 0 0))
+  )
+  (wire (pts (xy 195.58 83.82) (xy 208.28 83.82))
+    (stroke (width 0) (type default) (color 0 0 0 0))
+  )
+  (wire (pts (xy 195.58 129.54) (xy 177.8 129.54))
+    (stroke (width 0) (type default) (color 0 0 0 0))
+  )
+  (wire (pts (xy 177.8 93.98) (xy 180.34 93.98))
     (stroke (width 0) (type default) (color 0 0 0 0))
   )
@@
     (stroke (width 0) (type default) (color 0 0 0 0))
   )
+  (wire (pts (xy 186.69 88.9) (xy 186.69 106.68))
+    (stroke (width 0) (type default) (color 0 0 0 0))
+  )
   (wire (pts (xy 182.88 67.31) (xy 182.88 83.82))
     (stroke (width 0) (type default) (color 0 0 0 0))
@@
     (stroke (width 0) (type default) (color 0 0 0 0))
   )
+  (wire (pts (xy 186.69 106.68) (xy 195.58 106.68))
+    (stroke (width 0) (type default) (color 0 0 0 0))
+  )
   (wire (pts (xy 116.84 83.82) (xy 127 83.82))
     (stroke (width 0) (type default) (color 0 0 0 0))
@@
     (stroke (width 0) (type default) (color 0 0 0 0))
   )
+  (wire (pts (xy 180.34 93.98) (xy 180.34 99.06))
+    (stroke (width 0) (type default) (color 0 0 0 0))
+  )
   (wire (pts (xy 177.8 119.38) (xy 177.8 121.92))
     (stroke (width 0) (type default) (color 0 0 0 0))
   )
+  (wire (pts (xy 195.58 83.82) (xy 195.58 86.36))
+    (stroke (width 0) (type default) (color 0 0 0 0))
+  )
   (wire (pts (xy 127 83.82) (xy 132.08 83.82))
     (stroke (width 0) (type default) (color 0 0 0 0))
@@
     (stroke (width 0) (type default) (color 0 0 0 0))
   )
+  (wire (pts (xy 195.58 104.14) (xy 195.58 106.68))
+    (stroke (width 0) (type default) (color 0 0 0 0))
+  )
   (wire (pts (xy 116.84 101.6) (xy 104.14 101.6))
     (stroke (width 0) (type default) (color 0 0 0 0))
@@
     (stroke (width 0) (type default) (color 0 0 0 0))
   )
+  (wire (pts (xy 195.58 127) (xy 195.58 129.54))
+    (stroke (width 0) (type default) (color 0 0 0 0))
+  )
   (wire (pts (xy 134.62 81.28) (xy 132.08 81.28))
     (stroke (width 0) (type default) (color 0 0 0 0))
@@
     (stroke (width 0) (type default) (color 0 0 0 0))
   )
+  (wire (pts (xy 180.34 99.06) (xy 177.8 99.06))
+    (stroke (width 0) (type default) (color 0 0 0 0))
+  )
+  (wire (pts (xy 195.58 106.68) (xy 195.58 109.22))
+    (stroke (width 0) (type default) (color 0 0 0 0))
+  )
   (wire (pts (xy 104.14 129.54) (xy 104.14 130.81))
     (stroke (width 0) (type default) (color 0 0 0 0))
@@
   )
   (wire (pts (xy 116.84 99.06) (xy 116.84 101.6))
+    (stroke (width 0) (type default) (color 0 0 0 0))
+  )
+  (wire (pts (xy 177.8 88.9) (xy 186.69 88.9))
     (stroke (width 0) (type default) (color 0 0 0 0))
   )
@@
     (pin "2")
   )
-  (symbol (lib_id "power:+BATT") (at 101.6 83.82 90) (unit 1)
-    (in_bom yes) (on_board yes) (fields_autoplaced)
-    (property "Reference" "#PWR0105" (id 0) (at 105.41 83.82 0)
-      (effects (font (size 1.27 1.27)) hide)
-    )
-    (property "Value" "" (id 1) (at 97.79 83.8199 90)
-      (effects (font (size 1.27 1.27)) (justify left))
-    )
-    (property "Footprint" "" (id 2) (at 101.6 83.82 0)
-      (effects (font (size 1.27 1.27)) hide)
-    )
-    (property "Datasheet" "" (id 3) (at 101.6 83.82 0)
-      (effects (font (size 1.27 1.27)) hide)
-    )
+  (symbol (lib_id "CRCW040210K0FKED:CRCW040210K0FKED") (at 195.58 127 90) (unit 1)
+    (in_bom yes) (on_board yes) (fields_autoplaced)
+    (property "Reference" "R?" (id 0) (at 198.12 116.8399 90)
+      (effects (font (size 1.27 1.27)) (justify right))
+    )
+    (property "Value" "" (id 1) (at 198.12 119.3799 90)
+      (effects (font (size 1.27 1.27)) (justify right))
+    )
+    (property "Footprint" "" (id 2) (at 194.31 113.03 0)
+      (effects (font (size 1.27 1.27)) (justify left) hide)
+    )
+    (property "Datasheet" "http://www.vishay.com/docs/20035/dcrcwe3.pdf" (id 3) (at 196.85 113.03 0)
+      (effects (font (size 1.27 1.27)) (justify left) hide)
+    )
+    (property "Description" "CRCW0402 Resistor T/R 0.063W,1%,10K Vishay CRCW Series Thick Film Surface Mount Resistor 0402 Case 10k +/-1% 0.063W +/-100ppm/C" (id 4) (at 199.39 113.03 0)
+      (effects (font (size 1.27 1.27)) (justify left) hide)
+    )
+    (property "Height" "0.4" (id 5) (at 201.93 113.03 0)
+      (effects (font (size 1.27 1.27)) (justify left) hide)
+    )
+    (property "Mouser Part Number" "71-CRCW0402-10K-E3" (id 6) (at 204.47 113.03 0)
+      (effects (font (size 1.27 1.27)) (justify left) hide)
+    )
+    (property "Mouser Price/Stock" "https://www.mouser.co.uk/ProductDetail/Vishay-Dale/CRCW040210K0FKED?qs=rlE3Te1NifyN3e8vvxacSw%3D%3D" (id 7) (at 207.01 113.03 0)
+      (effects (font (size 1.27 1.27)) (justify left) hide)
+    )
+    (property "Manufacturer_Name" "Vishay" (id 8) (at 209.55 113.03 0)
+      (effects (font (size 1.27 1.27)) (justify left) hide)
+    )
+    (property "Manufacturer_Part_Number" "CRCW040210K0FKED" (id 9) (at 212.09 113.03 0)
+      (effects (font (size 1.27 1.27)) (justify left) hide)
+    )
+    (pin "1")
+    (pin "2")
+  )
+  (symbol (lib_id "CRCW040240K2FKED:CRCW040240K2FKED") (at 195.58 104.14 90) (unit 1)
+    (in_bom yes) (on_board yes) (fields_autoplaced)
+    (property "Reference" "R2" (id 0) (at 198.12 93.9799 90)
+      (effects (font (size 1.27 1.27)) (justify right))
+    )
+    (property "Value" "" (id 1) (at 198.12 96.5199 90)
+      (effects (font (size 1.27 1.27)) (justify right))
+    )
+    (property "Footprint" "" (id 2) (at 194.31 90.17 0)
+      (effects (font (size 1.27 1.27)) (justify left) hide)
+    )
+    (property "Datasheet" "http://www.vishay.com/docs/20035/dcrcwe3.pdf" (id 3) (at 196.85 90.17 0)
+      (effects (font (size 1.27 1.27)) (justify left) hide)
+    )
+    (property "Description" "CRCW0402 Resistor T/R 0.063W,1%,40K2 Vishay CRCW Series Thick Film Surface Mount Resistor 0402 Case 40.2k +/-1% 0.063W +/-100ppm/C" (id 4) (at 199.39 90.17 0)
+      (effects (font (size 1.27 1.27)) (justify left) hide)
+    )
+    (property "Height" "0.4" (id 5) (at 201.93 90.17 0)
+      (effects (font (size 1.27 1.27)) (justify left) hide)
+    )
+    (property "Mouser Part Number" "71-CRCW0402-40.2K-E3" (id 6) (at 204.47 90.17 0)
+      (effects (font (size 1.27 1.27)) (justify left) hide)
+    )
+    (property "Mouser Price/Stock" "https://www.mouser.co.uk/ProductDetail/Vishay-Dale/CRCW040240K2FKED?qs=rzhQWu8UUS3g49JmcwYN7w%3D%3D" (id 7) (at 207.01 90.17 0)
+      (effects (font (size 1.27 1.27)) (justify left) hide)
+    )
+    (property "Manufacturer_Name" "Vishay" (id 8) (at 209.55 90.17 0)
+      (effects (font (size 1.27 1.27)) (justify left) hide)
+    )
+    (property "Manufacturer_Part_Number" "CRCW040240K2FKED" (id 9) (at 212.09 90.17 0)
+      (effects (font (size 1.27 1.27)) (justify left) hide)
+    )
+    (pin "1")
+    (pin "2")
+  )
+  (symbol (lib_id "power:+BATT") (at 104.14 81.28 0) (unit 1)
+    (in_bom yes) (on_board yes) (fields_autoplaced)
+    (property "Reference" "#PWR0105" (id 0) (at 104.14 85.09 0)
+      (effects (font (size 1.27 1.27)) hide)
+    )
+    (property "Value" "" (id 1) (at 104.14 76.2 0))
+    (property "Footprint" "" (id 2) (at 104.14 81.28 0)
+      (effects (font (size 1.27 1.27)) hide)
+    )
+    (property "Datasheet" "" (id 3) (at 104.14 81.28 0)
+      (effects (font (size 1.27 1.27)) hide)
+    )
